File: real-eagle/real.sch (EAGLE design)
At the start: 18 parts, among them J2 POWER_JACK

Commit message: Schematic without layout
Parts:
- removed FET1: NEXFET_CSD18542KTT, real_library:NEXFET_CSD18542KTT
- removed P1, P2, P3, P4: (no value), real_library:NORCOMP_DUAL_PORT_DSUB9
Connections:
- net PWM0 renamed PWM_A0
- net PWM1 renamed PWM_A1
- net PWM10 renamed PWM_B2
- net PWM11 renamed PWM_B3
- net PWM12 renamed PWM_B4
- net PWM13 renamed PWM_B5
- net PWM14 renamed PWM_B6
- net PWM15 renamed PWM_B7
- net PWM16 renamed PWM_C0
- net PWM17 renamed PWM_C1
- net PWM18 renamed PWM_C2
- net PWM19 renamed PWM_C3
- net PWM2 renamed PWM_A2
- net PWM20 renamed PWM_C4
- net PWM21 renamed PWM_C5
- net PWM22 renamed PWM_C6
- net PWM23 renamed PWM_C7
- net PWM24 renamed PWM_D0
- net PWM25 renamed PWM_D1
- net PWM26 renamed PWM_D2
- net PWM27 renamed PWM_D3
- net PWM28 renamed PWM_D4
- net PWM29 renamed PWM_D5
- net PWM3 renamed PWM_A3
- net PWM30 renamed PWM_D6
- net PWM31 renamed PWM_D7
- net PWM4 renamed PWM_A4
- net PWM5 renamed PWM_A5
- net PWM6 renamed PWM_A6
- net PWM7 renamed PWM_A7
- net PWM8 renamed PWM_B0
- net PWM9 renamed PWM_B1
- removed net HEATER0: P1.P$1, P1.Q$1
- removed net HEATER1: P1.P$2, P1.Q$2
- removed net HEATER10: P2.P$3, P2.Q$3
- removed net HEATER11: P2.P$4, P2.Q$4
- removed net HEATER12: P2.P$5, P2.Q$5
- removed net HEATER13: P2.P$6, P2.Q$6
- removed net HEATER14: P2.P$7, P2.Q$7
- removed net HEATER15: P2.P$8, P2.Q$8
- removed net HEATER16: P3.P$1, P3.Q$1
- removed net HEATER17: P3.P$2, P3.Q$2
- removed net HEATER18: P3.P$3, P3.Q$3
- removed net HEATER19: P3.P$4, P3.Q$4
- removed net HEATER2: P1.P$3, P1.Q$3
- removed net HEATER20: P3.P$5, P3.Q$5
- removed net HEATER21: P3.P$6, P3.Q$6
- removed net HEATER22: P3.P$7, P3.Q$7
- removed net HEATER23: P3.P$8, P3.Q$8
- removed net HEATER24: P4.P$1, P4.Q$1
- removed net HEATER25: P4.P$2, P4.Q$2
- removed net HEATER26: P4.P$3, P4.Q$3
- removed net HEATER27: P4.P$4, P4.Q$4
- removed net HEATER28: P4.P$5, P4.Q$5
- removed net HEATER29: P4.P$6, P4.Q$6
- removed net HEATER3: P1.P$4, P1.Q$4
- removed net HEATER30: P4.P$7, P4.Q$7
- removed net HEATER31: P4.P$8, P4.Q$8
- removed net HEATER4: P1.P$5, P1.Q$5
- removed net HEATER5: P1.P$6, P1.Q$6
- removed net HEATER6: P1.P$7, P1.Q$7
- removed net HEATER7: P1.P$8, P1.Q$8
- removed net HEATER8: P2.P$1, P2.Q$1
- removed net HEATER9: P2.P$2, P2.Q$2
- net GND: no longer P1.P$9, P1.Q$9, P2.P$9, P2.Q$9, P3.P$9, P3.Q$9, P4.P$9, P4.Q$9
- net VCC: now also U2.VDD
