File: real-eagle/real_with_onsemi.sch (EAGLE design)
At the start: 13 parts, among them J2 POWER_JACK

Commit message: Add modifications from @slacAdpai as of 2019/2/27
Parts:
- removed JP_I2C: (no value), pinhead:PINHD-1X2
- added J_48V: PHOENIX_TERMINAL_BLOCK, real_library:PHOENIX_TERMINAL_BLOCK
- added TP_5V, TP_CANHI, TP_CANLO, TP_GND, TP_I2C+, TP_I2C-, TP_RS485A, TP_RS485B: TPB1,27, testpad:TPB1,27
- R_CAN, R_RS485: device rcl:R-US_0207/12 -> rcl:R-US_R1206; SPICEPREFIX 120 -> (none)
- R_SCL, R_SDA: value 4.7K -> 4.7k; device rcl:R-US_0207/12 -> rcl:R-US_R0805; SPICEPREFIX 120 -> (none)
Connections:
- new net V_48V: J_48V.1
- net GND: now also J_48V.2, TP_GND.TP
- net N$1: now also R_CAN.1, TP_CANLO.TP; no longer R_CAN.2
- net N$16: no longer JP_I2C.2
- net N$19: no longer JP_I2C.1
- net N$3: now also TP_CANHI.TP
- net N$4: now also R_CAN.2; no longer R_CAN.1
- net VCC: now also TP_5V.TP
Other:
- note added: "120Ω resistor P/N: HRG3216P-1200-D-T1"
- note added: "4.7kΩ resistor P/N: CRGCQ0805F4K7"
- note added: "48V 100A terminal block P/N: 1932588 Phoenix Contact"
- moved on the sheet: R_CAN
